File: rocket2-load-cell.kicad_pcb (KiCad board)
At the start: 2 copper layers, 42 x 53.5 mm, 34 parts, among them J1 SWD, J2 Screw_Terminal_01x02, U2 STM32F103C8Tx, U3 AMS1117-3.3, Y1 16MHz

Commit message: Revert "finished routing file(submit for review)"
This reverts commit a7b270876cc0567c9db231a326dac314d918e378.
Parts:
- removed H1, H2, H3, H4: MountingHole, MountingHole:MountingHole_3.2mm_M3
- added C10: 100nF, Capacitor_SMD:C_0603_1608Metric, F.Cu at (119.4, 99.8)
- added C12: 10uF, Capacitor_SMD:C_0603_1608Metric, F.Cu at (119.4, 104.9)
- added C15: 100nF, Capacitor_SMD:C_0603_1608Metric, F.Cu at (123.4, 97.3)
- moved J1 69.4 mm to (105.5, 64.5), turned to 90 degrees
- moved R4 68.9 mm to (104.0, 53.5)
- moved C20 68.7 mm to (101.5, 55.0), turned to 0 degrees
- moved JP1 68.6 mm to (115.5, 68.5)
- moved R2 68.4 mm to (104.0, 56.5)
- moved ADS1219 68.0 mm to (97.0, 56.5), turned to 90 degrees
- moved J2 66.9 mm to (115.5, 82.6)
- moved U3 65.5 mm to (105.5, 81.0)
- moved U1 65.3 mm to (92.9, 81.8)
- moved C5 64.7 mm to (88.5, 70.0)
- moved C8 64.5 mm to (88.5, 73.3), turned to -90 degrees
- moved Y1 64.4 mm to (84.8, 70.2), turned to 90 degrees
- moved C14 64.4 mm to (88.5, 66.8)
- moved C3 64.4 mm to (97.5, 76.0)
- moved C7 64.4 mm to (92.2, 64.0)
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Connections:
- ADS1219 pad 3: Net-(ADS1219-RESET) -> ADS_RESET
- C14 pad 1: +3.3V -> GND
- C14 pad 2: GND -> +3.3V
- JP1 pad 2: GND -> AIN+
- JP1 pad 3: Net-(C13-Pad1) -> AIN-
- JP1 pad 4: AIN- -> GND
- JP1 pad 5: AIN+ -> Net-(C13-Pad1)
- R3 pad 1: Net-(ADS1219-RESET) -> ADS_RESET
Routing:
- net +3.3V: track 146.4 -> 0.00 mm, vias 2 -> 0
- net GND: track 39.7 -> 0.00 mm, vias 11 -> 0
- net VBUS: track 25.8 -> 0.00 mm
- net NRST: track 19.4 -> 0.00 mm
- net MEM_WP: track 18.1 -> 0.00 mm, vias 2 -> 0
- net Net-(C13-Pad1): track 16.7 -> 0.00 mm
- net MEM_MISO: track 14.5 -> 0.00 mm, vias 2 -> 0
- net MEM_CS: track 14.5 -> 0.00 mm, vias 2 -> 0
- net DEBUG_SWDIO: track 12.5 -> 0.00 mm
- net ADS_DRDY: track 12.0 -> 0.00 mm
- net DEBUG_SWCLK: track 9.96 -> 0.00 mm
- net ADS_DATA: track 7.84 -> 0.00 mm
- net AIN-: track 7.68 -> 0.00 mm
- net ADS_CLK: track 6.95 -> 0.00 mm
- net AIN+: track 6.95 -> 0.00 mm
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- removed copper zone on B.Cu, net GND
Other:
- board outline removed
