File: rocket2-load-cell.kicad_pcb (KiCad board)
At the start: 2 copper layers, 69 x 67 mm, 38 parts, among them J1 SWD, J2 Screw_Terminal_01x02, U2 STM32F103C8Tx, U3 AMS1117-3.3, Y1 16MHz

Commit message: added code and stab
Parts:
- added R6: 2.2K, Resistor_SMD:R_0603_1608Metric, F.Cu at (140.5, 102.5)
- added R7: 2.2K, Resistor_SMD:R_0603_1608Metric, F.Cu at (135.7, 102.0)
Routing:
- net +3.3V: track 210.4 -> 214.6 mm
