File: rocket2-load-cell.kicad_sch (KiCad schematic)
At the start: 34 parts, among them J1 SWD, J2 Screw_Terminal_01x02, U2 STM32F103C8Tx, U3 AMS1117-3.3, Y1 16MHz

Commit message: Revert "finished routing file(submit for review)"
This reverts commit a7b270876cc0567c9db231a326dac314d918e378.
Parts:
- removed H1, H2, H3, H4: MountingHole, MountingHole:MountingHole_3.2mm_M3, symbol Mechanical:MountingHole
- added C10, C15: 100nF, Capacitor_SMD:C_0603_1608Metric, symbol Device:C_Small
- added C12: 10uF, Capacitor_SMD:C_0603_1608Metric, symbol Device:C_Small
Connections:
- net +3.3V: now also C10.1, C12.1, C15.1
- net ADS_RESET: now also ADS1219.3 (RESET), R3.1
- net AIN+: now also JP1.2; no longer JP1.5
- net AIN-: now also JP1.3; no longer JP1.4
- net GND: now also JP1.4, C10.2, C12.2, C15.2; no longer JP1.2
- net at C13.1, C18.1, L2.1: now also JP1.5; no longer JP1.3
Other:
- note removed: "Made to use standard M3 screws"
- moved on the sheet: C13, C18, L2
